File: pcb/Ventilator/Ventilator.kicad_pcb (KiCad board)
At the start: 2 copper layers, 103 x 86.5 mm, 79 parts, among them J1 Conn_02x03_Top_Bottom, J3 Screw_Terminal_01x02, J4 Screw_Terminal_01x03, J5 Screw_Terminal_01x02, K1 FINDER-40.52.7.012.0000, Q1 NUD3160, Q2 NUD3160, Q3 NUD3160, SW1 Reset, U1 Pico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

Commit message: - last changes
Parts:
- R3: moved to B.Cu
- moved D6 2.30 mm to (107.1, 120.7)
- moved PS1 1.73 mm to (129.5, 167.1)
- moved C10 1.40 mm to (133.6, 168.5)
- moved R1 1.02 mm to (87.9, 172.2)
- moved D1 1.02 mm to (86.9, 182.0)
- moved J1 0.78 mm to (125.1, 121.8)
- moved U6 0.66 mm to (113.3, 120.5)
- moved C9 0.63 mm to (128.0, 168.5)
Routing:
- net GND: track 348.8 -> 377.0 mm, vias 31 -> 24
- net Net-(R3-Pad1): track 35.6 -> 59.3 mm
- net Net-(R13-Pad1): track 35.5 -> 13.6 mm, vias 1 -> 0
- net +12V: track 248.3 -> 230.4 mm, vias 1 -> 3
- net /CPU/SWCLK: track 52.9 -> 64.7 mm
- net +3.3V: track 150.5 -> 139.4 mm, vias 1 -> 0
- net Net-(R26-Pad1): track 25.1 -> 14.2 mm
- net Net-(C3-Pad1): track 12.3 -> 2.53 mm
- net /CPU/SWD: track 61.3 -> 67.1 mm
- net /CPU/IN1: track 94.7 -> 99.2 mm
- net /CPU/IN2: track 82.9 -> 78.8 mm
- net /CPU/IN3: track 68.9 -> 66.3 mm
- net +5V: track 25.0 -> 27.6 mm
- net Net-(D1-Pad1): track 66.8 -> 69.3 mm
- net /CPU/SCNN: track 37.6 -> 35.4 mm, vias 1 -> 0
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Other:
- board text added: "L"
- board text added: "SP2"
- board text added: "SP3"
- board text added: "VAK"
