File: pcb/Ventilator/Ventilator.kicad_pcb (KiCad board)
At the start: 2 copper layers, 103 x 86.5 mm, 79 parts, among them J1 Conn_02x03_Top_Bottom, J3 Screw_Terminal_01x02, J4 Screw_Terminal_01x03, J5 Screw_Terminal_01x02, K1 FINDER-40.52.7.012.0000, Q1 NUD3160, Q2 NUD3160, Q3 NUD3160, SW1 Reset, U1 Pico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

Commit message: - as ordered
Parts:
- D12: value BAT760,115 -> S07M-M-08
- moved Q1 2.70 mm to (113.0, 120.5)
- turned D6 to 90 degrees
Connections:
- U6 pad 1: Net-(D6-Pad2) -> +12V
- U6 pad 3: unconnected-(U6-Pad3) -> Net-(J3-Pad1)
- U6 pad 4: unconnected-(U6-Pad4) -> Net-(J3-Pad2)
- U6 pad 8: +12V -> Net-(D6-Pad2)
Routing:
- net /CPU/IN2: track 78.8 -> 113.8 mm
- net Net-(R3-Pad1): track 59.3 -> 39.0 mm, vias 0 -> 1
- net GND: track 377.0 -> 359.0 mm, vias 24 -> 32
- net /CPU/IN4: track 51.5 -> 63.4 mm
- net /CPU/IN1: track 99.2 -> 110.3 mm
- net +3.3V: track 139.4 -> 149.3 mm, vias 0 -> 1
- net Net-(C3-Pad1): track 2.53 -> 12.3 mm
- net Net-(R13-Pad1): track 13.6 -> 23.1 mm, vias 0 -> 1
- net Net-(J3-Pad2): track 17.8 -> 24.4 mm
- net Net-(J3-Pad1): track 15.0 -> 21.6 mm
- net Net-(D6-Pad2): track 24.1 -> 18.8 mm
- net /CPU/IN3: track 66.3 -> 71.4 mm
- net /CPU/SCLK: track 31.2 -> 35.8 mm
- net /CPU/RX: track 19.3 -> 22.8 mm
- net Net-(D12-Pad2): track 5.79 -> 8.76 mm
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Other:
- board text added: "Ventcontrol 1.3"
- board text removed: "Ventcontrol 1.2"
