File: pcb/Ventilator/Power.kicad_sch (KiCad schematic)
At the start: 7 parts, among them J4 Screw_Terminal_01x02, U7 NCP1117-3.3_SOT223

Commit message: - all parts connected, placed partially
Parts:
- renumbered C23 to C22, C24 to C23, C25 to C24, C26 to C25
Connections:
- net +12V: now reaches C22.1, J4.2 (Pin_2), PS1.1 (+VIN), PS1.2 (+VIN)
Changed lines of the file:
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@@
+    (stroke (width 0) (type default) (color 0 0 0 0))
+  )
+  (wire (pts (xy 74.93 77.47) (xy 74.93 81.28))
     (stroke (width 0) (type default) (color 0 0 0 0))
   )
@@
     (effects (font (size 1.27 1.27)) (justify left bottom))
   )
+  (symbol (lib_id "power:+12V") (at 74.93 77.47 0) (unit 1)
+    (in_bom yes) (on_board yes) (fields_autoplaced)
+    (property "Reference" "#PWR0106" (id 0) (at 74.93 81.28 0)
+      (effects (font (size 1.27 1.27)) hide)
+    )
+    (property "Value" "+12V" (id 1) (at 74.93 72.39 0))
+    (property "Footprint" "" (id 2) (at 74.93 77.47 0)
+      (effects (font (size 1.27 1.27)) hide)
+    )
+    (property "Datasheet" "" (id 3) (at 74.93 77.47 0)
+      (effects (font (size 1.27 1.27)) hide)
+    )
+    (pin "1")
+  )
   (symbol (lib_id "Device:C") (at 140.97 92.71 0) (unit 1)
     (in_bom yes) (on_board yes) (fields_autoplaced)
-    (property "Reference" "C25" (id 0) (at 144.78 91.4399 0)
+    (property "Reference" "C24" (id 0) (at 144.78 91.4399 0)
       (effects (font (size 1.27 1.27)) (justify left))
     )
@@
   (symbol (lib_id "Device:C") (at 74.93 92.71 0) (unit 1)
     (in_bom yes) (on_board yes) (fields_autoplaced)
-    (property "Reference" "C23" (id 0) (at 78.74 91.4399 0)
+    (property "Reference" "C22" (id 0) (at 78.74 91.4399 0)
       (effects (font (size 1.27 1.27)) (justify left))
     )
@@
   (symbol (lib_id "Device:C") (at 120.65 92.71 0) (unit 1)
     (in_bom yes) (on_board yes) (fields_autoplaced)
-    (property "Reference" "C24" (id 0) (at 124.46 91.4399 0)
+    (property "Reference" "C23" (id 0) (at 124.46 91.4399 0)
       (effects (font (size 1.27 1.27)) (justify left))
     )
@@
   (symbol (lib_id "power:VCC") (at 120.65 77.47 0) (unit 1)
     (in_bom yes) (on_board yes) (fields_autoplaced)
-    (property "Reference" "#PWR028" (id 0) (at 120.65 81.28 0)
+    (property "Reference" "#PWR030" (id 0) (at 120.65 81.28 0)
       (effects (font (size 1.27 1.27)) hide)
     )
@@
   (symbol (lib_id "Device:C") (at 172.72 92.71 0) (unit 1)
     (in_bom yes) (on_board yes) (fields_autoplaced)
-    (property "Reference" "C26" (id 0) (at 176.53 91.4399 0)
+    (property "Reference" "C25" (id 0) (at 176.53 91.4399 0)
       (effects (font (size 1.27 1.27)) (justify left))
     )
@@
   (symbol (lib_id "power:+3.3V") (at 176.53 77.47 0) (unit 1)
     (in_bom yes) (on_board yes) (fields_autoplaced)
-    (property "Reference" "#PWR029" (id 0) (at 176.53 81.28 0)
+    (property "Reference" "#PWR031" (id 0) (at 176.53 81.28 0)
       (effects (font (size 1.27 1.27)) hide)
     )
@@
   (symbol (lib_id "power:GND") (at 106.68 102.87 0) (unit 1)
     (in_bom yes) (on_board yes) (fields_autoplaced)
-    (property "Reference" "#PWR027" (id 0) (at 106.68 109.22 0)
+    (property "Reference" "#PWR029" (id 0) (at 106.68 109.22 0)
       (effects (font (size 1.27 1.27)) hide)
     )
@@
   (symbol (lib_id "power:GND") (at 99.06 102.87 0) (unit 1)
     (in_bom yes) (on_board yes) (fields_autoplaced)
-    (property "Reference" "#PWR026" (id 0) (at 99.06 109.22 0)
-      (effects (font (size 1.27 1.27)) hide)
-    )
+    (property "Reference" "#PWR028" (id 0) (at 99.06 109.22 0)
+      (effects (font (size 1.27 1.27)) hide)
+    )

Commit message: - voor omschakeling naar rp pico
Parts:
- added D12: BAT760,115, Diode_SMD:D_SOD-323_HandSoldering, symbol Device:D_Schottky
- renumbered C22 to C21, C23 to C22, C24 to C23, C25 to C24, U7 to U8
Connections:
- net +12V: now also D12.1 (K); no longer J4.2 (Pin_2)
- new net: D12.2 (A), J4.2 (Pin_2)
Other:
- moved on the sheet: J4
Changed lines of the file:
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@@
   (junction (at 74.93 81.28) (diameter 0) (color 0 0 0 0)
+  )
+  (junction (at 113.03 102.87) (diameter 0) (color 0 0 0 0)
   )
   (junction (at 120.65 81.28) (diameter 0) (color 0 0 0 0)
@@
   (no_connect (at 114.3 86.36))
   (no_connect (at 83.82 86.36))
+  (wire (pts (xy 53.34 81.28) (xy 60.96 81.28))
+    (stroke (width 0) (type default) (color 0 0 0 0))
+  )
   (wire (pts (xy 67.31 102.87) (xy 74.93 102.87))
     (stroke (width 0) (type default) (color 0 0 0 0))
@@
     (stroke (width 0) (type default) (color 0 0 0 0))
   )
-  (wire (pts (xy 64.77 83.82) (xy 67.31 83.82))
+  (wire (pts (xy 53.34 83.82) (xy 67.31 83.82))
     (stroke (width 0) (type default) (color 0 0 0 0))
   )
@@
     (stroke (width 0) (type default) (color 0 0 0 0))
   )
-  (wire (pts (xy 106.68 102.87) (xy 115.57 102.87))
+  (wire (pts (xy 106.68 102.87) (xy 113.03 102.87))
     (stroke (width 0) (type default) (color 0 0 0 0))
   )
@@
     (stroke (width 0) (type default) (color 0 0 0 0))
   )
+  (wire (pts (xy 113.03 102.87) (xy 115.57 102.87))
+    (stroke (width 0) (type default) (color 0 0 0 0))
+  )
   (wire (pts (xy 140.97 96.52) (xy 140.97 102.87))
     (stroke (width 0) (type default) (color 0 0 0 0))
@@
     (stroke (width 0) (type default) (color 0 0 0 0))
   )
-  (wire (pts (xy 64.77 81.28) (xy 74.93 81.28))
-    (stroke (width 0) (type default) (color 0 0 0 0))
-  )
   (wire (pts (xy 165.1 81.28) (xy 172.72 81.28))
     (stroke (width 0) (type default) (color 0 0 0 0))
@@
   )
   (wire (pts (xy 120.65 102.87) (xy 140.97 102.87))
+    (stroke (width 0) (type default) (color 0 0 0 0))
+  )
+  (wire (pts (xy 68.58 81.28) (xy 74.93 81.28))
     (stroke (width 0) (type default) (color 0 0 0 0))
   )
@@
   (symbol (lib_id "power:+12V") (at 74.93 77.47 0) (unit 1)
     (in_bom yes) (on_board yes) (fields_autoplaced)
-    (property "Reference" "#PWR0106" (id 0) (at 74.93 81.28 0)
+    (property "Reference" "#PWR031" (id 0) (at 74.93 81.28 0)
       (effects (font (size 1.27 1.27)) hide)
     )
@@
   (symbol (lib_id "Device:C") (at 140.97 92.71 0) (unit 1)
     (in_bom yes) (on_board yes) (fields_autoplaced)
-    (property "Reference" "C24" (id 0) (at 144.78 91.4399 0)
+    (property "Reference" "C23" (id 0) (at 144.78 91.4399 0)
       (effects (font (size 1.27 1.27)) (justify left))
     )
@@
   (symbol (lib_id "Device:C") (at 74.93 92.71 0) (unit 1)
     (in_bom yes) (on_board yes) (fields_autoplaced)
-    (property "Reference" "C22" (id 0) (at 78.74 91.4399 0)
+    (property "Reference" "C21" (id 0) (at 78.74 91.4399 0)
       (effects (font (size 1.27 1.27)) (justify left))
     )
@@
   (symbol (lib_id "Device:C") (at 120.65 92.71 0) (unit 1)
     (in_bom yes) (on_board yes) (fields_autoplaced)
-    (property "Reference" "C23" (id 0) (at 124.46 91.4399 0)
+    (property "Reference" "C22" (id 0) (at 124.46 91.4399 0)
       (effects (font (size 1.27 1.27)) (justify left))
     )
@@
   (symbol (lib_id "power:VCC") (at 120.65 77.47 0) (unit 1)
     (in_bom yes) (on_board yes) (fields_autoplaced)
-    (property "Reference" "#PWR030" (id 0) (at 120.65 81.28 0)
+    (property "Reference" "#PWR034" (id 0) (at 120.65 81.28 0)
       (effects (font (size 1.27 1.27)) hide)
     )
@@
   (symbol (lib_id "Device:C") (at 172.72 92.71 0) (unit 1)
     (in_bom yes) (on_board yes) (fields_autoplaced)
-    (property "Reference" "C25" (id 0) (at 176.53 91.4399 0)
+    (property "Reference" "C24" (id 0) (at 176.53 91.4399 0)
       (effects (font (size 1.27 1.27)) (justify left))
     )
@@
   (symbol (lib_id "power:+3.3V") (at 176.53 77.47 0) (unit 1)
     (in_bom yes) (on_board yes) (fields_autoplaced)
-    (property "Reference" "#PWR031" (id 0) (at 176.53 81.28 0)
+    (property "Reference" "#PWR035" (id 0) (at 176.53 81.28 0)
       (effects (font (size 1.27 1.27)) hide)
     )
@@
   (symbol (lib_id "power:GND") (at 106.68 102.87 0) (unit 1)
     (in_bom yes) (on_board yes) (fields_autoplaced)
-    (property "Reference" "#PWR029" (id 0) (at 106.68 109.22 0)
+    (property "Reference" "#PWR033" (id 0) (at 106.68 109.22 0)
       (effects (font (size 1.27 1.27)) hide)
     )
@@
   (symbol (lib_id "Regulator_Linear:NCP1117-3.3_SOT223") (at 157.48 81.28 0) (unit 1)
     (in_bom yes) (on_board yes) (fields_autoplaced)
-    (property "Reference" "U7" (id 0) (at 157.48 73.66 0))
+    (property "Reference" "U8" (id 0) (at 157.48 73.66 0))
     (property "Value" "NCP1117-3.3_SOT223" (id 1) (at 157.48 76.2 0))
     (property "Footprint" "Package_TO_SOT_SMD:SOT-223-3_TabPin2" (id 2) (at 157.48 76.2 0)
@@
   (symbol (lib_id "power:GND") (at 99.06 102.87 0) (unit 1)
     (in_bom yes) (on_board yes) (fields_autoplaced)
-    (property "Reference" "#PWR028" (id 0) (at 99.06 109.22 0)
+    (property "Reference" "#PWR032" (id 0) (at 99.06 109.22 0)
       (effects (font (size 1.27 1.27)) hide)
     )
@@
     (pin "1")
   )
-  (symbol (lib_id "Connector:Screw_Terminal_01x02") (at 59.69 83.82 180) (unit 1)
-    (in_bom yes) (on_board yes) (fields_autoplaced)
-    (property "Reference" "J4" (id 0) (at 59.69 74.93 0))
-    (property "Value" "Screw_Terminal_01x02" (id 1) (at 59.69 77.47 0))
-    (property "Footprint" "TerminalBlock:TerminalBlock_bornier-2_P5.08mm" (id 2) (at 59.69 83.82 0)
-      (effects (font (size 1.27 1.27)) hide)
-    )
-    (property "Datasheet" "~" (id 3) (at 59.69 83.82 0)
-      (effects (font (size 1.27 1.27)) hide)
-    )
-    (pin "1")
-    (pin "2")
+  (symbol (lib_id "Connector:Screw_Terminal_01x02") (at 48.26 83.82 180) (unit 1)
+    (in_bom yes) (on_board yes) (fields_autoplaced)
+    (property "Reference" "J4" (id 0) (at 48.26 74.93 0))
+    (property "Value" "Screw_Terminal_01x02" (id 1) (at 48.26 77.47 0))
+    (property "Footprint" "TerminalBlock:TerminalBlock_bornier-2_P5.08mm" (id 2) (at 48.26 83.82 0)
+      (effects (font (size 1.27 1.27)) hide)
+    )
+    (property "Datasheet" "~" (id 3) (at 48.26 83.82 0)
+      (effects (font (size 1.27 1.27)) hide)
+    )
+    (pin "1")
+    (pin "2")
+  )
+  (symbol (lib_id "Device:D_Schottky") (at 64.77 81.28 180) (unit 1)
+    (in_bom yes) (on_board yes) (fields_autoplaced)
+    (property "Reference" "D12" (id 0) (at 65.0875 74.93 0))
+    (property "Value" "BAT760,115" (id 1) (at 65.0875 77.47 0))
+    (property "Footprint" "Diode_SMD:D_SOD-323_HandSoldering" (id 2) (at 64.77 81.28 0)
+      (effects (font (size 1.27 1.27)) hide)
+    )
+    (property "Datasheet" "~" (id 3) (at 64.77 81.28 0)
+      (effects (font (size 1.27 1.27)) hide)
+    )
+    (pin "1")
+    (pin "2")
+  )
+  (symbol (lib_id "power:PWR_FLAG") (at 113.03 102.87 180) (unit 1)
+    (in_bom yes) (on_board yes) (fields_autoplaced)
+    (property "Reference" "#FLG01" (id 0) (at 113.03 104.775 0)
+      (effects (font (size 1.27 1.27)) hide)
+    )
+    (property "Value" "PWR_FLAG" (id 1) (at 115.57 104.1399 0)
+      (effects (font (size 1.27 1.27)) (justify right))
+    )
+    (property "Footprint" "" (id 2) (at 113.03 102.87 0)
+      (effects (font (size 1.27 1.27)) hide)
+    )
+    (property "Datasheet" "~" (id 3) (at 113.03 102.87 0)
+      (effects (font (size 1.27 1.27)) hide)
+    )
+    (pin "1")
   )
 )

Commit message: - voor autorouter
Parts:
- removed C23, C24: 10u, Capacitor_SMD:C_0805_2012Metric_Pad1.18x1.45mm_HandSolder, symbol Device:C
- removed U8: NCP1117-3.3_SOT223, Package_TO_SOT_SMD:SOT-223-3_TabPin2, symbol Regulator_Linear:NCP1117-3.3_SOT223
- PS1: value R-78AA3.3-0.5SMD-R -> R-78AA5.0-0.5SMD-R
- renumbered C22 to C10, C21 to C9
Connections:
- net VCC renamed +5V

Commit message: -Ventcontrol 1.2 (routed)
Parts:
- D12: footprint Diode_SMD:D_SOD-323_HandSoldering -> Diode_SMD:D_SMF
- renumbered J4 to J5
Changed lines of the file:
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@@
   (symbol (lib_id "Connector:Screw_Terminal_01x02") (at 48.26 83.82 180) (unit 1)
     (in_bom yes) (on_board yes) (fields_autoplaced)
-    (property "Reference" "J4" (id 0) (at 48.26 74.93 0))
+    (property "Reference" "J5" (id 0) (at 48.26 74.93 0))
     (property "Value" "Screw_Terminal_01x02" (id 1) (at 48.26 77.47 0))
     (property "Footprint" "TerminalBlock:TerminalBlock_bornier-2_P5.08mm" (id 2) (at 48.26 83.82 0)
@@
     (property "Reference" "D12" (id 0) (at 65.0875 74.93 0))
     (property "Value" "BAT760,115" (id 1) (at 65.0875 77.47 0))
-    (property "Footprint" "Diode_SMD:D_SOD-323_HandSoldering" (id 2) (at 64.77 81.28 0)
+    (property "Footprint" "Diode_SMD:D_SMF" (id 2) (at 64.77 81.28 0)
       (effects (font (size 1.27 1.27)) hide)
     )

Commit message: - as ordered
Parts:
- D12: value BAT760,115 -> S07M-M-08
Changed lines of the file:
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@@
     (in_bom yes) (on_board yes) (fields_autoplaced)
     (property "Reference" "D12" (id 0) (at 65.0875 74.93 0))
-    (property "Value" "BAT760,115" (id 1) (at 65.0875 77.47 0))
+    (property "Value" "S07M-M-08" (id 1) (at 65.0875 77.47 0))
     (property "Footprint" "Diode_SMD:D_SMF" (id 2) (at 64.77 81.28 0)
       (effects (font (size 1.27 1.27)) hide)
